File: pcb/adidas.kicad_pcb (KiCad board)
At the start: 2 copper layers, 152.7 x 107.2 mm, 34 parts, among them J1 ISP Header, J2 Shitty Add-on, J4 Battery, U1 MPU-6050, U2 ATTINY841-SSU

Commit message: update the battery clip in the BOM
Parts:
- removed REF**: MountingHole_4.5mm, DEAD10C5:MountingHole_4.5mm
- BT1: value Battery_Cell -> Battery Clip
Changed lines of the file:
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@@
     )
-  )
-  (footprint "DEAD10C5:MountingHole_4.5mm" (layer "F.Cu")
-    (at 165.0492 48.2092)
-    (descr "Mounting Hole 4.5mm, no annular")
-    (tags "mounting hole 4.5mm no annular")
-    (attr exclude_from_pos_files exclude_from_bom)
-    (fp_text reference "REF**" (at 0 -5.5) (layer "F.SilkS") hide
-        (effects (font (size 1 1) (thickness 0.15)))
-    )
-    (fp_text value "MountingHole_4.5mm" (at 0 5.5) (layer "F.Fab") hide
-        (effects (font (size 1 1) (thickness 0.15)))
-    )
-    (fp_text user "${REFERENCE}" (at 0 0) (layer "F.Fab") hide
-        (effects (font (size 1 1) (thickness 0.15)))
-    )
-    (fp_circle (center 0 0) (end 4.5 0)
-      (stroke (width 0.15) (type solid)) (fill none) (layer "Cmts.User"))
-    (fp_circle (center 0 0) (end 4.75 0)
-      (stroke (width 0.05) (type solid)) (fill none) (layer "F.CrtYd"))
-    (pad "" np_thru_hole circle (at 0 0) (size 4.5 4.5) (drill 4.5) (layers "*.Cu" "*.Mask"))
   )
   (footprint "LED_SMD:LED_1206_3216Metric" (layer "F.Cu")
@@
     (property "Color" "White")
     (property "Digi-Key Part Number" "2679-CTL1206FWH1TTR-ND")
-    (property "MANUFACTURER" "Venkel")
     (property "MAXIMUM_PACKAGE_HEIGHT" "1.2mm")
+    (property "Manufacturer" "Venkel")
     (property "STANDARD" "Manufacturer Recommendations")
     (property "Sheetfile" "adidas.kicad_sch")
@@
     (descr "https://www.tme.eu/it/Document/a823211ec201a9e209042d155fe22d2b/KEYS2996.pdf")
     (tags "BR2016 CR2016 DL2016 BR2020 CL2020 BR2025 CR2025 DL2025 DR2032 CR2032 DL2032")
-    (property "Sheetfile" "adidas.kicad_sch")
-    (property "Sheetname" "")
+    (property "Description" "CR2032 Coin Cell Battery Holder")
+    (property "Manufacturer" "Keystone Electronics")
+    (property "Manufacturer Product Number" "3000TR")
+    (property "Mouser Part Number`" "534-3000TR")
+    (property "Sheetfile" "adidas.kicad_sch")
+    (property "Sheetname" "")
+    (property "exclude_from_bom" "")
     (property "ki_description" "Single-cell battery")
     (property "ki_keywords" "battery cell")
-    (attr smd)
+    (attr smd exclude_from_bom)
     (fp_text reference "BT1" (at -9.15 -9.7) (layer "B.SilkS") hide
         (effects (font (size 1 1) (thickness 0.15)) (justify mirror))
     )
-    (fp_text value "Battery_Cell" (at 0 11) (layer "B.Fab") hide
+    (fp_text value "Battery Clip" (at 0 11) (layer "B.Fab") hide
         (effects (font (size 1 1) (thickness 0.15)) (justify mirror))
     )
@@
   (footprint "DEAD10C5:QFN50P400X400X95-24N" (layer "B.Cu")
     (at 165.481 99.2378 180)
-    (property "AVAILABILITY" "Good")
     (property "DESCRIPTION" "IMU ACCEL/GYRO 3-AXIS I2C 24QFN")
     (property "Description" "IMU ACCEL/GYRO 3-AXIS I2C 24QFN")
-    (property "MF" "TDK")
     (property "MP" "MPU-6050")
     (property "Manufacturer" "TDK")
@@
     (property "Mouser Part " "410-MPU-6050")
     (property "PACKAGE" "QFN-24 InvenSense")
-    (property "PARTREV" "3.4")
-    (property "PRICE" "5.45 USD")
-    (property "STANDARD" "IPC-7351B")
-    (property "Sheetfile" "adidas.kicad_sch")
-    (property "Sheetname" "")
+    (property "Sheetfile" "adidas.kicad_sch")
+    (property "Sheetname" "")
