File: v3/adidas.kicad_pcb (KiCad board)
At the start: 2 copper layers, 152.7 x 107.2 mm, 36 parts, among them J1 ISP Header, J2 Shitty Add-on, J4 Battery, U1 MPU-6050, U2 ATTINY841-SSU

Commit message: random checkpoint (#44)
* random checkpoint

* redo routing on PCB

* refactor a bit

* more moounting holes

* tune up reuse

* tune up reuse

* update names
Parts:
- added hole-left: MountingHole_4.5mm, DEAD10C5:MountingHole_4.5mm, F.Cu at (234.6, 76.2)
- added hole-right: MountingHole_4.5mm, DEAD10C5:MountingHole_4.5mm, F.Cu at (96.6, 76.6)
- J4: value Battery -> батарея
- moved S2 2.14 mm to (234.6, 86.9)
- renumbered REF** to hole1
Routing:
- net GND: track 0.00 -> 391.3 mm, vias 0 -> 3
- net VDD: track 0.00 -> 199.8 mm
- net /9(SCK): track 0.00 -> 174.1 mm, vias 0 -> 2
- net /7(SDA): track 0.00 -> 162.4 mm, vias 0 -> 2
- net /4(RST): track 0.00 -> 159.6 mm
- net /13(SAO1): track 0.00 -> 116.6 mm
- net /8(MOSI): track 0.00 -> 113.8 mm, vias 0 -> 1
- net /12(SAO2): track 0.00 -> 93.0 mm, vias 0 -> 1
- net /3(LED Mid Row): track 0.00 -> 89.6 mm
- net /5(LED Top Row): track 0.00 -> 78.2 mm
- net Net-(D1-Pad2): track 0.00 -> 75.2 mm, vias 0 -> 1
- net Net-(D8-Pad2): track 0.00 -> 61.7 mm, vias 0 -> 1
- net Net-(D7-Pad2): track 0.00 -> 57.9 mm, vias 0 -> 1
- net Net-(D12-Pad2): track 0.00 -> 55.7 mm, vias 0 -> 1
- net /2(LED Bottom Row): track 0.00 -> 54.6 mm
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Other:
- board text added: ":: THE @DEAD10C5 LOVE YOU :: justinjustin yaya_pancho @craigmucka Hermit y3t1 @p0lr_ @thedevilsvoice"
- board text removed: ":: THE @DEAD10C5 LOVE YOU :: @p0lr_ Eddie the Yeti yaya_pancho @thedevilsvoice"
